File: cardshark.kicad_sch (KiCad schematic)
At the start: 93 parts, among them J1 Conn_02x03_Odd_Even, J2 Bus_ISA_8bit, J3 DE15_Receptacle_HighDensity_M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, U1 LM334M, U10 SN74F260DR, U11 93CxxA, U12 SOJ_256Kx16, U13 SOJ_256Kx16, U14 27C010, U2 GD543x_VLB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

Commit message: Add files via upload
Big bunch'o little minor fixes, no version number change (mostly to clean up libraries and eliminate a bunch of previously silenced ERC warnings)
Parts:
- removed U1: LM334M, Package_SO:SOIC-8_3.9x4.9mm_P1.27mm, symbol Reference_Current:LM334M
- removed U14: 27C010, PLCC-32:PLCC-32_SMD-Socket, symbol Memory_EPROM:27C010
- added U5: 27C010, PDVGA:PLCC-32_SMD-Socket, symbol PDVGA:27C010
- added U9: LM334M, PDVGA:SOIC-8_DMP-8, symbol PDVGA:LM334M
- R10, R29, R30, R7, R8, R9: footprint Resistor_SMD:R_0603_1608Metric -> Resistor_SMD:R_0805_2012Metric
- RN2: footprint Resistor_SMD:R_Array_Convex_4x0603 -> PDVGA:ResArray_Convex_4x0603
- U11: footprint Package_SO:SOIC-8_3.9x4.9mm_P1.27mm -> PDVGA:SOIC-8_DMP-8
- U12, U13, U3, U7: footprint SOJ_DRAM:SOJ-40_10.16x26.44mm_P1.27mm -> PDVGA:SOJ-40_10.16x26.44mm_P1.27mm; symbol SOJ_DRAM:SOJ_256Kx16 -> PDVGA:SOJ_256Kx16
Connections:
- net A15: now also U5.3 (A15)
- net A16: now also U5.2 (A16)
- net BD0: now also U5.13 (D0)
- net BD1: now also U5.14 (D1)
- net BD2: now also U5.15 (D2)
- net BD3: now also U5.17 (D3)
- net BD4: now also U5.18 (D4)
- net BD5: now also U5.19 (D5)
- net BD6: now also U5.20 (D6)
- net BD7: now also U5.21 (D7)
- net EROM: now also U5.22 (~{CE})
- net GND: now also U5.16 (GND)
- net IREF: now also U9.4
- net SA0: now also U5.12 (A0)
- net SA1: now also U5.11 (A1)
- net SA10: now also U5.23 (A10)
- net SA11: now also U5.25 (A11)
- net SA12: now also U5.4 (A12)
- net SA13: now also U5.28 (A13)
- net SA14: now also U5.29 (A14)
- net SA2: now also U5.10 (A2)
- net SA3: now also U5.9 (A3)
- net SA4: now also U5.8 (A4)
- net SA5: now also U5.7 (A5)
- net SA6: now also U5.6 (A6)
- net SA7: now also U5.5 (A7)
- net SA8: now also U5.27 (A8)
- net SA9: now also U5.26 (A9)
- net VCC: now also U5.32 (VCC)
- net ~{SMEMRD}: now also U5.24 (~{OE})
- net at D1.2 (A), R32.2: now also U9.2, U9.3, U9.6, U9.7
- net at R31.2, R32.1: now also U9.1
- net ADR27: no longer names the net of U8.B24 (A27)
- net ADR28: no longer names the net of U8.A22 (A28)
- net ADR29: no longer names the net of U8.B23 (A29)
- net ADR30: no longer names the net of U8.A21 (A30)
Other:
- note added: "Unfiltered Mode: Omit C27-C32, replace FB1-3 with 0 ohm resistors"
- note removed: "Happy Tiido Mode: Omit C27-C32, replace FB1-3 with 0 ohm resistors"
